File: STM32MP1_Processor.kicad_sch (KiCad schematic)
At the start: 6 parts, among them U1 STM32MP131DAFx

Commit message: Initial Connections
Initial Draw
Parts:
- added R10, R11, R12, R13, R14, R16, R17, R6, R7, R8, R9: 33R, symbol Device:R
Connections:
- net at U1.A15 (PB9): now also R11.2
- net at U1.A16 (PF0): now also R10.2
- net at U1.B14 (PC6): now also R12.2
- net at U1.B15 (PB15): now also R7.2
- net at U1.B16 (PB14): now also R6.2
- net at U1.B17 (PE3): now also R17.2
- net at U1.C13 (PC7): now also R13.2
- net at U1.C14 (PB3): now also R8.2
- net at U1.C16 (PB4): now also R9.2
- net at U1.C17 (PG6): now also R14.2
- net at U1.G2 (PG10): now also R16.2
- new net eMMC_CLK: R17.1
- new net eMMC_CMD: R14.1
- new net eMMC_DATA6: R12.1
- new net eMMC_RST: R16.1
