File: DDR3_RAM.kicad_sch (KiCad schematic)
At the start: 8 parts, among them U3 AS4C256M16D3

Commit message: added mmc schematic
Parts:
- added C10, C11, C12, C15, C16, C17, C4, C5, C6: 100nF, Capacitor_SMD:C_0402_1005Metric, symbol Device:C_Small
- added C13, C14, C18, C19, C7, C8, C9: 10uF, Capacitor_SMD:C_0805_2012Metric, symbol Device:C_Small
- added R30: 100R, Resistor_SMD:R_0402_1005Metric, symbol Device:R_Small
Connections:
- net CK_N: now also R30.2
- net CK_P: now also R30.1
- net GND: now also C10.2, C11.2, C12.2, C13.2, C14.2, C15.2, C16.2, C17.2, C18.2, C19.2, C4.2, C5.2, C6.2, C7.2, C8.2, C9.2
- net VDD_DDR: now also C10.1, C11.1, C12.1, C13.1, C14.1, C15.1, C16.1, C17.1, C18.1, C19.1, C4.1, C5.1, C6.1, C7.1, C8.1, C9.1

Commit message: Updated Processor With ETH Pins
Also updated Capacitors and Resistors to 402
Parts:
- C13, C14, C18, C19, C7, C8, C9: footprint Capacitor_SMD:C_0805_2012Metric -> Capacitor_SMD:C_0402_1005Metric
Changed lines of the file:
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@@
 			)
 		)
-		(property "Footprint" "Capacitor_SMD:C_0805_2012Metric"
+		(property "Footprint" "Capacitor_SMD:C_0402_1005Metric"
 			(at 80.01 68.58 0)
 			(effects
@@
 			)
 		)
-		(property "Footprint" "Capacitor_SMD:C_0805_2012Metric"
+		(property "Footprint" "Capacitor_SMD:C_0402_1005Metric"
 			(at 80.01 27.94 0)
 			(effects
@@
 			)
 		)
-		(property "Footprint" "Capacitor_SMD:C_0805_2012Metric"
+		(property "Footprint" "Capacitor_SMD:C_0402_1005Metric"
 			(at 40.64 48.26 0)
 			(effects
@@
 			)
 		)
-		(property "Footprint" "Capacitor_SMD:C_0805_2012Metric"
+		(property "Footprint" "Capacitor_SMD:C_0402_1005Metric"
 			(at 40.64 68.58 0)
 			(effects
@@
 			)
 		)
-		(property "Footprint" "Capacitor_SMD:C_0805_2012Metric"
+		(property "Footprint" "Capacitor_SMD:C_0402_1005Metric"
 			(at 40.64 27.94 0)
 			(effects
@@
 			)
 		)
-		(property "Footprint" "Capacitor_SMD:C_0805_2012Metric"
+		(property "Footprint" "Capacitor_SMD:C_0402_1005Metric"
 			(at 80.01 48.26 0)
 			(effects
@@
 			)
 		)
-		(property "Footprint" "Capacitor_SMD:C_0805_2012Metric"
+		(property "Footprint" "Capacitor_SMD:C_0402_1005Metric"
 			(at 88.9 48.26 0)
 			(effects
