File: EMMC.kicad_sch (KiCad schematic)
At the start: 23 parts, among them U2 EMMC04G-S100-B08U

Commit message: Included Tushar's changed also added SDCARD module
Parts:
- added C24, C30: 10uF, Capacitor_SMD:C_0805_2012Metric, symbol Device:C_Small
- added C25, C26, C27: 100nF, Capacitor_SMD:C_0402_1005Metric, symbol Device:C_Small
- added C28: 100nF, Capacitor_SMD:C_0805_2012Metric, symbol Device:C_Small
- added C29: 2.2uF, Capacitor_SMD:C_0805_2012Metric, symbol Device:C_Small
- added R43, R44: 0R, Resistor_SMD:R_0402_1005Metric, symbol Device:R_Small
Connections:
- net EMMC_3V3: now also C24.1, C25.1, C26.1, C27.1, C28.1, R43.1, R44.1
- net EMMC_CLK: now also C30.1
- net GND: now also C24.2, C25.2, C26.2, C27.2, C28.2, C29.2, C30.2
- net at U2.C2 (VDDI): now also C29.1
- new net SYS_3V3: R44.2
- new net VDD_EMMC: R43.2
Other:
- moved on the sheet: R29

Commit message: Updated Processor With ETH Pins
Also updated Capacitors and Resistors to 402
Parts:
- C24, C28, C29, C30: footprint Capacitor_SMD:C_0805_2012Metric -> Capacitor_SMD:C_0402_1005Metric
Changed lines of the file:
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@@
 			)
 		)
-		(property "Footprint" "Capacitor_SMD:C_0805_2012Metric"
+		(property "Footprint" "Capacitor_SMD:C_0402_1005Metric"
 			(at 118.11 148.59 0)
 			(effects
@@
 			)
 		)
-		(property "Footprint" "Capacitor_SMD:C_0805_2012Metric"
+		(property "Footprint" "Capacitor_SMD:C_0402_1005Metric"
 			(at 78.74 148.59 0)
 			(effects
@@
 			)
 		)
-		(property "Footprint" "Capacitor_SMD:C_0805_2012Metric"
+		(property "Footprint" "Capacitor_SMD:C_0402_1005Metric"
 			(at 149.86 110.49 0)
 			(effects
@@
 			)
 		)
-		(property "Footprint" "Capacitor_SMD:C_0805_2012Metric"
+		(property "Footprint" "Capacitor_SMD:C_0402_1005Metric"
 			(at 181.61 81.28 0)
 			(effects
