File: Ethernet.kicad_sch (KiCad schematic)
At the start: 46 parts, among them U4 LAN8742A

Commit message: Temporary changes
My changes
Connections:
- net TXEN is gone; now on net REFCLK0: R57.1
Other:
- moved on the sheet: R55, R56, R57, R58, R59, R60, R61
Changed lines of the file:
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@@
 	(wire
 		(pts
-			(xy 109.22 71.12) (xy 134.62 71.12)
+			(xy 111.76 71.12) (xy 134.62 71.12)
 		)
 		(stroke
@@
 	(wire
 		(pts
-			(xy 109.22 78.74) (xy 134.62 78.74)
+			(xy 111.76 78.74) (xy 134.62 78.74)
 		)
 		(stroke
@@
 	(wire
 		(pts
-			(xy 109.22 83.82) (xy 134.62 83.82)
+			(xy 111.76 83.82) (xy 134.62 83.82)
 		)
 		(stroke
@@
 	(wire
 		(pts
-			(xy 109.22 76.2) (xy 134.62 76.2)
+			(xy 111.76 76.2) (xy 134.62 76.2)
 		)
 		(stroke
@@
 	(wire
 		(pts
-			(xy 96.52 86.36) (xy 104.14 86.36)
+			(xy 99.06 86.36) (xy 106.68 86.36)
 		)
 		(stroke
@@
 	(wire
 		(pts
-			(xy 109.22 81.28) (xy 134.62 81.28)
+			(xy 111.76 81.28) (xy 134.62 81.28)
 		)
 		(stroke
@@
 	(wire
 		(pts
-			(xy 96.52 81.28) (xy 104.14 81.28)
+			(xy 99.06 81.28) (xy 106.68 81.28)
 		)
 		(stroke
@@
 	(wire
 		(pts
-			(xy 96.52 73.66) (xy 104.14 73.66)
+			(xy 99.06 73.66) (xy 106.68 73.66)
 		)
 		(stroke
@@
 	(wire
 		(pts
-			(xy 96.52 83.82) (xy 104.14 83.82)
+			(xy 99.06 83.82) (xy 106.68 83.82)
 		)
 		(stroke
@@
 	(wire
 		(pts
-			(xy 96.52 71.12) (xy 104.14 71.12)
+			(xy 99.06 71.12) (xy 106.68 71.12)
 		)
 		(stroke
@@
 	(wire
 		(pts
-			(xy 109.22 86.36) (xy 134.62 86.36)
+			(xy 111.76 86.36) (xy 134.62 86.36)
 		)
 		(stroke
@@
 	(wire
 		(pts
-			(xy 109.22 73.66) (xy 134.62 73.66)
+			(xy 111.76 73.66) (xy 134.62 73.66)
 		)
 		(stroke
@@
 	(wire
 		(pts
-			(xy 96.52 78.74) (xy 104.14 78.74)
+			(xy 99.06 78.74) (xy 106.68 78.74)
 		)
 		(stroke
@@
 	(wire
 		(pts
-			(xy 96.52 76.2) (xy 104.14 76.2)
+			(xy 99.06 76.2) (xy 106.68 76.2)
 		)
 		(stroke
@@
 		)
 	)
-	(label "ETH9"
+	(label "ETH0"
 		(at 44.45 123.19 180)
 		(effects
@@
 	(hierarchical_label "RXD1"
 		(shape input)
-		(at 96.52 81.28 180)
+		(at 99.06 81.28 180)
 		(effects
 			(font
@@
 	(hierarchical_label "TXD0"
 		(shape input)
-		(at 96.52 71.12 180)
+		(at 99.06 71.12 180)
 		(effects
 			(font
@@
 	(hierarchical_label "RXD0"
 		(shape input)
-		(at 96.52 78.74 180)
+		(at 99.06 78.74 180)
 		(effects
 			(font
@@
 	(hierarchical_label "TXEN"
 		(shape input)
-		(at 96.52 76.2 180)
+		(at 99.06 76.2 180)
 		(effects
 			(font
@@
 	(hierarchical_label "CRX_DV"
 		(shape input)
-		(at 96.52 86.36 180)
+		(at 99.06 86.36 180)
 		(effects
 			(font
@@
 	(hierarchical_label "VCC"
 		(shape input)
-		(at 96.52 83.82 180)
+		(at 99.06 83.82 180)
 		(effects
 			(font
@@
 	(hierarchical_label "TXD1"
 		(shape input)
-		(at 96.52 73.66 180)
+		(at 99.06 73.66 180)
 		(effects
 			(font
@@
 	(symbol
 		(lib_id "Device:R_Small")
-		(at 106.68 86.36 90)
+		(at 109.22 86.36 90)
 		(unit 1)
 		(exclude_from_sim no)
@@
 		(dnp no)
 		(property "Reference" "R60"
-			(at 102.362 85.344 90)
+			(at 104.902 85.344 90)
 			(effects
 				(font
@@
 		)
 		(property "Value" "33R"
-			(at 110.49 85.09 90)
+			(at 113.03 85.09 90)
 			(effects
 				(font
@@
 		)
 		(property "Footprint" "Resistor_SMD:R_0402_1005Metric"
-			(at 106.68 86.36 0)
+			(at 109.22 86.36 0)
 			(effects
 				(font
@@
 		)
 		(property "Datasheet" "~"
-			(at 106.68 86.36 0)
+			(at 109.22 86.36 0)
 			(effects
 				(font
@@
 		)
 		(property "Description" "Resistor, small symbol"
-			(at 106.68 86.36 0)
+			(at 109.22 86.36 0)
 			(effects
 				(font
@@
 	(symbol
 		(lib_id "Device:R_Small")
-		(at 106.68 81.28 90)
+		(at 109.22 81.28 90)
 		(unit 1)
 		(exclude_from_sim no)
@@
 		(dnp no)
 		(property "Reference" "R59"
-			(at 102.362 80.264 90)
+			(at 104.902 80.264 90)
 			(effects
 				(font
@@
 		)
 		(property "Value" "33R"
-			(at 110.49 80.01 90)
+			(at 113.03 80.01 90)
 			(effects
 				(font
@@
 		)
 		(property "Footprint" "Resistor_SMD:R_0402_1005Metric"
-			(at 106.68 81.28 0)
+			(at 109.22 81.28 0)
 			(effects
 				(font
@@
 		)
 		(property "Datasheet" "~"
-			(at 106.68 81.28 0)
+			(at 109.22 81.28 0)
 			(effects
 				(font
@@
 		)
 		(property "Description" "Resistor, small symbol"
-			(at 106.68 81.28 0)
+			(at 109.22 81.28 0)
 			(effects
 				(font
@@
 	(symbol
 		(lib_id "Device:R_Small")
-		(at 106.68 76.2 90)
+		(at 109.22 76.2 90)
 		(unit 1)
 		(exclude_from_sim no)
@@
 		(dnp no)
 		(property "Reference" "R57"
-			(at 102.362 75.184 90)
+			(at 104.902 75.184 90)
 			(effects
 				(font
@@
 		)
 		(property "Value" "33R"
-			(at 110.49 74.93 90)
+			(at 113.03 74.93 90)
 			(effects
 				(font
@@
 		)
 		(property "Footprint" "Resistor_SMD:R_0402_1005Metric"
-			(at 106.68 76.2 0)
+			(at 109.22 76.2 0)
 			(effects
 				(font
@@
 		)
 		(property "Datasheet" "~"
-			(at 106.68 76.2 0)
+			(at 109.22 76.2 0)
 			(effects
 				(font
@@
 		)
 		(property "Description" "Resistor, small symbol"
-			(at 106.68 76.2 0)
+			(at 109.22 76.2 0)
 			(effects
 				(font
@@
 	(symbol
 		(lib_id "Device:R_Small")
-		(at 106.68 78.74 90)
+		(at 109.22 78.74 90)
 		(unit 1)
 		(exclude_from_sim no)
@@
 		(dnp no)
 		(property "Reference" "R58"
-			(at 102.362 77.724 90)
+			(at 104.902 77.724 90)
 			(effects
 				(font
@@
 		)
 		(property "Value" "33R"
-			(at 110.49 77.47 90)
+			(at 113.03 77.47 90)
 			(effects
 				(font
@@
 		)
 		(property "Footprint" "Resistor_SMD:R_0402_1005Metric"
-			(at 106.68 78.74 0)
+			(at 109.22 78.74 0)
 			(effects
 				(font
@@
 		)
 		(property "Datasheet" "~"
-			(at 106.68 78.74 0)
+			(at 109.22 78.74 0)
 			(effects
 				(font
@@
 		)
 		(property "Description" "Resistor, small symbol"
-			(at 106.68 78.74 0)
+			(at 109.22 78.74 0)
 			(effects
 				(font
@@
 	(symbol
 		(lib_id "Device:R_Small")
-		(at 106.68 83.82 90)
+		(at 109.22 83.82 90)
 		(unit 1)
 		(exclude_from_sim no)
@@
 		(dnp no)
 		(property "Reference" "R61"
-			(at 102.362 82.804 90)
+			(at 104.902 82.804 90)
 			(effects
 				(font
@@
 		)
 		(property "Value" "10R"
-			(at 110.49 82.55 90)
+			(at 113.03 82.55 90)
 			(effects
 				(font
@@
 		)
 		(property "Footprint" "Resistor_SMD:R_0402_1005Metric"
-			(at 106.68 83.82 0)
+			(at 109.22 83.82 0)
 			(effects
 				(font
@@
 		)
 		(property "Datasheet" "~"
-			(at 106.68 83.82 0)
+			(at 109.22 83.82 0)
 			(effects
 				(font
@@
 		)
 		(property "Description" "Resistor, small symbol"
-			(at 106.68 83.82 0)
+			(at 109.22 83.82 0)
 			(effects
 				(font
@@
 	(symbol
 		(lib_id "Device:R_Small")
-		(at 106.68 71.12 90)
+		(at 109.22 71.12 90)
 		(unit 1)
 		(exclude_from_sim no)
@@
 		(dnp no)
 		(property "Reference" "R56"
-			(at 102.362 70.104 90)
+			(at 104.902 70.104 90)
 			(effects
 				(font
@@
 		)
 		(property "Value" "33R"
-			(at 110.49 69.85 90)
+			(at 113.03 69.85 90)
 			(effects
 				(font
@@
 		)
 		(property "Footprint" "Resistor_SMD:R_0402_1005Metric"
-			(at 106.68 71.12 0)
+			(at 109.22 71.12 0)
 			(effects
 				(font
@@
 		)
 		(property "Datasheet" "~"
-			(at 106.68 71.12 0)
+			(at 109.22 71.12 0)
 			(effects
 				(font
@@
 		)
 		(property "Description" "Resistor, small symbol"
-			(at 106.68 71.12 0)
+			(at 109.22 71.12 0)
 			(effects
 				(font
@@
 	(symbol
 		(lib_id "Device:R_Small")
-		(at 106.68 73.66 90)
+		(at 109.22 73.66 90)
 		(unit 1)
 		(exclude_from_sim no)
@@
 		(dnp no)
 		(property "Reference" "R55"
-			(at 102.362 72.644 90)
+			(at 104.902 72.644 90)
 			(effects
 				(font
@@
 		)
 		(property "Value" "33R"
-			(at 110.49 72.39 90)
+			(at 113.03 72.39 90)
 			(effects
 				(font
@@
 		)
 		(property "Footprint" "Resistor_SMD:R_0402_1005Metric"
-			(at 106.68 73.66 0)
+			(at 109.22 73.66 0)
 			(effects
 				(font
@@
 		)
 		(property "Datasheet" "~"
-			(at 106.68 73.66 0)
+			(at 109.22 73.66 0)
 			(effects
 				(font
@@
 		)
 		(property "Description" "Resistor, small symbol"
-			(at 106.68 73.66 0)
+			(at 109.22 73.66 0)
 			(effects
 				(font
