File: eMMC.kicad_sch (KiCad schematic)
At the start: 3 parts, among them U2 EMMC04G-S100-B08U

Commit message: First
Parts:
- C4: value C -> 10 pf; footprint (none) -> Capacitor_SMD:C_0402_1005Metric
- C5: value C -> 2.2 uf; footprint (none) -> Capacitor_SMD:C_0603_1608Metric

Commit message: Temporary changes
My changes
Parts:
- removed C4: 10 pf, Capacitor_SMD:C_0402_1005Metric, symbol Device:C
- removed C5: 2.2 uf, Capacitor_SMD:C_0603_1608Metric, symbol Device:C
- added C24, C30: 10uF, Capacitor_SMD:C_0805_2012Metric, symbol Device:C_Small
- added C25, C26, C27: 100nF, Capacitor_SMD:C_0402_1005Metric, symbol Device:C_Small
- added C28: 100nF, Capacitor_SMD:C_0805_2012Metric, symbol Device:C_Small
- added C29: 2.2uF, Capacitor_SMD:C_0805_2012Metric, symbol Device:C_Small
- added R10, R11, R12, R13, R14, R15, R16, R27, R7, R8, R9: 33R, Resistor_SMD:R_0402_1005Metric, symbol Device:R_Small
- added R17, R18, R19, R20, R21, R22, R23, R24, R25, R29, R6: 10K, Resistor_SMD:R_0402_1005Metric, symbol Device:R_Small
- added R43, R44: 0R, Resistor_SMD:R_0402_1005Metric, symbol Device:R_Small
Connections:
- net GND: now also U2.A7 (RFU@1), C24.2, C25.2, C26.2, C27.2, C28.2, C29.2, C30.2
- net at U2.C2 (VDDI): now also C29.1
- net +3V3 renamed EMMC_3V3
- net EMMC_3V3: now also C24.1, C25.1, C26.1, C27.1, C28.1, R17.2, R18.2, R19.2, R20.2, R21.1, R22.1, R23.1, R24.1, R25.1, R29.1, R43.1, R44.1, R6.2
- net eMMC_CLK renamed EMMC_CLK
- net EMMC_CLK: now also C30.1, R16.2, R25.2
- net eMMC_CMD renamed EMMC_CMD
- net EMMC_CMD: now also R15.2, R24.2
- net eMMC_DATA0 renamed EMMC_DATA0
- net EMMC_DATA0: now also R6.1, R7.2
- net eMMC_DATA1 renamed EMMC_DATA1
- net EMMC_DATA1: now also R17.1, R8.2
- net eMMC_DATA2 renamed EMMC_DATA2
- net EMMC_DATA2: now also R18.1, R9.2
- net eMMC_DATA3 renamed EMMC_DATA3
- net EMMC_DATA3: now also R10.2, R19.1
- net eMMC_DATA4 renamed EMMC_DATA4
- net EMMC_DATA4: now also R11.2, R20.1
- net eMMC_DATA5 renamed EMMC_DATA5
- net EMMC_DATA5: now also R12.2, R21.2
- net eMMC_DATA6 renamed EMMC_DATA6
- net EMMC_DATA6: now also R13.2, R22.2
- net eMMC_DATA7 renamed EMMC_DATA7
- net EMMC_DATA7: now also R14.2, R23.2
- net eMMC_RST renamed ~{SYS_RST}
- net ~{SYS_RST}: now also R27.2, R29.2
- new net EMMC0: R7.1
- new net EMMC1: R8.1
- new net EMMC10: R27.1
- new net EMMC2: R9.1
- new net EMMC3: R10.1
- new net EMMC4: R11.1
- new net EMMC5: R12.1
- new net EMMC6: R13.1
- new net EMMC7: R14.1
- new net EMMC8: R15.1
- new net EMMC9: R16.1
- new net SYS_3V3: R44.2
- new net VDD_EMMC: R43.2
- no-connect marks 0 -> 11
Other:
- moved on the sheet: U2
