File: STM32MP1.kicad_pcb (KiCad board)
At the start: 2 copper layers, 15 parts, among them U1 STM32MP131DAFx, U2 EMMC04G-S100-B08U, U3 AS4C256M16D3

Commit message: added mmc schematic
Parts:
- added J1: Micro_SD_Card_Det1, microSD:J_SD_Card-micro_socket_A, F.Cu at (166.5, 93.5)
- added R10: 33R, Resistor_SMD:R_0402_1005Metric, F.Cu at (121.9, 125.8)
- added R11: 33R, Resistor_SMD:R_0402_1005Metric, F.Cu at (121.9, 127.8)
- added R12: 33R, Resistor_SMD:R_0402_1005Metric, F.Cu at (121.9, 129.8)
- added R13: 33R, Resistor_SMD:R_0402_1005Metric, F.Cu at (124.8, 117.9)
- added R14: 33R, Resistor_SMD:R_0402_1005Metric, F.Cu at (124.8, 119.8)
- added R15: 33R, Resistor_SMD:R_0402_1005Metric, F.Cu at (124.8, 121.8)
- added R16: 33R, Resistor_SMD:R_0402_1005Metric, F.Cu at (124.8, 123.8)
- added R17: 10K, Resistor_SMD:R_0402_1005Metric, F.Cu at (124.8, 125.8)
- added R18: 10K, Resistor_SMD:R_0402_1005Metric, F.Cu at (124.8, 127.8)
- added R19: 10K, Resistor_SMD:R_0402_1005Metric, F.Cu at (124.8, 129.8)
- added R20: 10K, Resistor_SMD:R_0402_1005Metric, F.Cu at (127.7, 117.9)
- added R21: 10K, Resistor_SMD:R_0402_1005Metric, F.Cu at (127.7, 119.8)
- added R22: 10K, Resistor_SMD:R_0402_1005Metric, F.Cu at (127.7, 121.8)
- added R23: 10K, Resistor_SMD:R_0402_1005Metric, F.Cu at (127.7, 123.8)
- added R24: 10K, Resistor_SMD:R_0402_1005Metric, F.Cu at (127.7, 125.8)
- added R25: 10K, Resistor_SMD:R_0402_1005Metric, F.Cu at (127.7, 127.8)
- added R26: 33R, Resistor_SMD:R_0402_1005Metric, F.Cu at (127.7, 129.8)
- added R27: 33R, Resistor_SMD:R_0402_1005Metric, F.Cu at (130.6, 117.9)
- added R28: 10K, Resistor_SMD:R_0402_1005Metric, F.Cu at (130.6, 119.8)
- added R29: 10K, Resistor_SMD:R_0402_1005Metric, F.Cu at (130.6, 121.8)
- added R6: 10K, Resistor_SMD:R_0402_1005Metric, F.Cu at (121.9, 117.9)
- added R7: 33R, Resistor_SMD:R_0402_1005Metric, F.Cu at (121.9, 119.8)
- added R8: 33R, Resistor_SMD:R_0402_1005Metric, F.Cu at (121.9, 121.8)
- added R9: 33R, Resistor_SMD:R_0402_1005Metric, F.Cu at (121.9, 123.8)
- moved U2 35.5 mm to (118.7, 107.0), turned to 90 degrees
- moved U1 5.52 mm to (113.5, 83.5)
- moved U3 2.53 mm to (129.5, 82.5)
Connections:
- C1 pad 1: /DDR3_RAM/VREF_DDR -> /STM32MP1_Processor/VDD_DDR
- C2 pad 1: /DDR3_RAM/VREF_DDR -> /STM32MP1_Processor/VDD_DDR
- C3 pad 2: /STM32MP1_Processor/GND -> /DDR3_RAM/GND
- R4 pad 1: /DDR3_RAM/VDD_DDR -> /STM32MP1_Processor/VDD_DDR
- R5 pad 2: /STM32MP1_Processor/GND -> /DDR3_RAM/GND
- U1 pad A1: /STM32MP1_Processor/GND -> /DDR3_RAM/GND
- U1 pad A15: unconnected-(U1-PB9-PadA15) -> /EMMC/EMMC5
- U1 pad A16: unconnected-(U1-PF0-PadA16) -> /EMMC/EMMC4
- U1 pad A21: /STM32MP1_Processor/GND -> /DDR3_RAM/GND
- U1 pad AA1: /STM32MP1_Processor/GND -> /DDR3_RAM/GND
- U1 pad AA18: /STM32MP1_Processor/GND -> /DDR3_RAM/GND
- U1 pad AA21: /STM32MP1_Processor/GND -> /DDR3_RAM/GND
- U1 pad B12: /STM32MP1_Processor/GND -> /DDR3_RAM/GND
- U1 pad B14: unconnected-(U1-PC6-PadB14) -> /EMMC/EMMC6
- U1 pad B15: unconnected-(U1-PB15-PadB15) -> /EMMC/EMMC1
- U1 pad B16: unconnected-(U1-PB14-PadB16) -> /EMMC/EMMC0
- U1 pad B17: unconnected-(U1-PE3-PadB17) -> /EMMC/EMMC9
- U1 pad C13: unconnected-(U1-PC7-PadC13) -> /EMMC/EMMC7
- U1 pad C14: unconnected-(U1-PB3-PadC14) -> /EMMC/EMMC2
- U1 pad C16: unconnected-(U1-PB4-PadC16) -> /EMMC/EMMC3
- U1 pad C17: unconnected-(U1-PG6-PadC17) -> /EMMC/EMMC8
- U1 pad D16: /STM32MP1_Processor/GND -> /DDR3_RAM/GND
- U1 pad E11: /STM32MP1_Processor/GND -> /DDR3_RAM/GND
- U1 pad E16: /STM32MP1_Processor/GND -> /DDR3_RAM/GND
- U1 pad E5: /STM32MP1_Processor/GND -> /DDR3_RAM/GND
- U1 pad E6: /STM32MP1_Processor/GND -> /DDR3_RAM/GND
- U1 pad F17: /STM32MP1_Processor/GND -> /DDR3_RAM/GND
- U1 pad F18: /STM32MP1_Processor/GND -> /DDR3_RAM/GND
- U1 pad F21: /STM32MP1_Processor/GND -> /DDR3_RAM/GND
- U1 pad F5: /STM32MP1_Processor/GND -> /DDR3_RAM/GND
- U1 pad G12: /STM32MP1_Processor/GND -> /DDR3_RAM/GND
- U1 pad G14: /STM32MP1_Processor/GND -> /DDR3_RAM/GND
- U1 pad G8: /STM32MP1_Processor/GND -> /DDR3_RAM/GND
- U1 pad H15: /STM32MP1_Processor/GND -> /DDR3_RAM/GND
- U1 pad H7: /STM32MP1_Processor/GND -> /DDR3_RAM/GND
- U1 pad J10: /STM32MP1_Processor/GND -> /DDR3_RAM/GND
- U1 pad J12: /STM32MP1_Processor/GND -> /DDR3_RAM/GND
- U1 pad K1: /STM32MP1_Processor/GND -> /DDR3_RAM/GND
- U1 pad K10: /STM32MP1_Processor/GND -> /DDR3_RAM/GND
- U1 pad K11: /STM32MP1_Processor/GND -> /DDR3_RAM/GND
- U1 pad K12: /STM32MP1_Processor/GND -> /DDR3_RAM/GND
- U1 pad K13: /STM32MP1_Processor/GND -> /DDR3_RAM/GND
- U1 pad K21: /STM32MP1_Processor/GND -> /DDR3_RAM/GND
- U1 pad K9: /STM32MP1_Processor/GND -> /DDR3_RAM/GND
- U1 pad L10: /STM32MP1_Processor/GND -> /DDR3_RAM/GND
- U1 pad L12: /STM32MP1_Processor/GND -> /DDR3_RAM/GND
- U1 pad L15: /STM32MP1_Processor/GND -> /DDR3_RAM/GND
- U1 pad L17: /STM32MP1_Processor/GND -> /DDR3_RAM/GND
- U1 pad L5: /STM32MP1_Processor/GND -> /DDR3_RAM/GND
- U1 pad M1: /STM32MP1_Processor/GND -> /DDR3_RAM/GND
- U1 pad M10: /STM32MP1_Processor/GND -> /DDR3_RAM/GND
- U1 pad M11: /STM32MP1_Processor/GND -> /DDR3_RAM/GND
- U1 pad M12: /STM32MP1_Processor/GND -> /DDR3_RAM/GND
- U1 pad M13: /STM32MP1_Processor/GND -> /DDR3_RAM/GND
- U1 pad M7: /STM32MP1_Processor/GND -> /DDR3_RAM/GND
- U1 pad M9: /STM32MP1_Processor/GND -> /DDR3_RAM/GND
- U1 pad N11: /STM32MP1_Processor/GND -> /DDR3_RAM/GND
- U1 pad P15: /STM32MP1_Processor/GND -> /DDR3_RAM/GND
- U1 pad P7: /STM32MP1_Processor/GND -> /DDR3_RAM/GND
- U1 pad R11: /STM32MP1_Processor/GND -> /DDR3_RAM/GND
- U1 pad R14: /STM32MP1_Processor/GND -> /DDR3_RAM/GND
- U1 pad R8: /STM32MP1_Processor/GND -> /DDR3_RAM/GND
- U1 pad T1: /STM32MP1_Processor/GND -> /DDR3_RAM/GND
- U1 pad T17: /STM32MP1_Processor/GND -> /DDR3_RAM/GND
- U1 pad T21: /STM32MP1_Processor/GND -> /DDR3_RAM/GND
- U1 pad T5: /STM32MP1_Processor/GND -> /DDR3_RAM/GND
- U1 pad U11: /STM32MP1_Processor/GND -> /DDR3_RAM/GND
- U1 pad U13: /STM32MP1_Processor/GND -> /DDR3_RAM/GND
- U1 pad U16: /STM32MP1_Processor/GND -> /DDR3_RAM/GND
- U1 pad U3: /STM32MP1_Processor/GND -> /DDR3_RAM/GND
- U1 pad U5: /STM32MP1_Processor/GND -> /DDR3_RAM/GND
- U1 pad U6: /STM32MP1_Processor/GND -> /DDR3_RAM/GND
- U1 pad U9: /STM32MP1_Processor/GND -> /DDR3_RAM/GND
- U1 pad V16: /STM32MP1_Processor/GND -> /DDR3_RAM/GND
- U1 pad W16: /STM32MP1_Processor/GND -> /DDR3_RAM/GND
- U1 pad Y11: unconnected-(U1-NRST-PadY11) -> /EMMC/EMMC11
- U1 pad Y14: /STM32MP1_Processor/GND -> /DDR3_RAM/GND
- U2 pad A3: unconnected-(U2-DAT0-PadA3) -> /EMMC/EMMC_DATA0
- U2 pad A4: unconnected-(U2-DAT1-PadA4) -> /EMMC/EMMC_DATA1
- U2 pad A5: unconnected-(U2-DAT2-PadA5) -> /EMMC/EMMC_DATA2
- U2 pad A6: unconnected-(U2-VSS1-PadA6) -> /EMMC/GND
- U2 pad A7: unconnected-(U2-RFU@1-PadA7) -> /EMMC/GND
- U2 pad B2: unconnected-(U2-DAT3-PadB2) -> /EMMC/EMMC_DATA3
- U2 pad B3: unconnected-(U2-DAT4-PadB3) -> /EMMC/EMMC_DATA4
- U2 pad B4: unconnected-(U2-DAT5-PadB4) -> /EMMC/EMMC_DATA5
- U2 pad B5: unconnected-(U2-DAT6-PadB5) -> /EMMC/EMMC_DATA6
- U2 pad B6: unconnected-(U2-DAT7-PadB6) -> /EMMC/EMMC_DATA7
- U2 pad C4: unconnected-(U2-VSSQ1-PadC4) -> /EMMC/GND
- U2 pad C6: unconnected-(U2-VCCQ1-PadC6) -> /EMMC/EMMC_3V3
- U2 pad E6: unconnected-(U2-VCC1-PadE6) -> /EMMC/EMMC_3V3
- U2 pad E7: unconnected-(U2-VSS2-PadE7) -> /EMMC/GND
- U2 pad F5: unconnected-(U2-VCC2-PadF5) -> /EMMC/EMMC_3V3
- U2 pad G5: unconnected-(U2-VSS3-PadG5) -> /EMMC/GND
- U2 pad H10: unconnected-(U2-VSS4-PadH10) -> /EMMC/GND
- U2 pad H5: unconnected-(U2-DS-PadH5) -> /EMMC/EMMC_DS
- U2 pad J10: unconnected-(U2-VCC3-PadJ10) -> /EMMC/EMMC_3V3
- U2 pad J5: unconnected-(U2-VSS5-PadJ5) -> /EMMC/GND
- U2 pad K5: unconnected-(U2-RST#-PadK5) -> /EMMC/~{SYS_RST}
- U2 pad K8: unconnected-(U2-VSS6-PadK8) -> /EMMC/GND
- U2 pad K9: unconnected-(U2-VCC4-PadK9) -> /EMMC/EMMC_3V3
- U2 pad M4: unconnected-(U2-VCCQ2-PadM4) -> /EMMC/EMMC_3V3
- U2 pad M5: unconnected-(U2-CMD-PadM5) -> /EMMC/EMMC_CMD
- U2 pad M6: unconnected-(U2-CLK-PadM6) -> /EMMC/EMMC_CLK
- U2 pad N2: unconnected-(U2-VSSQ2-PadN2) -> /EMMC/GND
- U2 pad N4: unconnected-(U2-VCCQ3-PadN4) -> /EMMC/EMMC_3V3
- U2 pad N5: unconnected-(U2-VSSQ3-PadN5) -> /EMMC/GND
- U2 pad P3: unconnected-(U2-VCCQ4-PadP3) -> /EMMC/EMMC_3V3
- U2 pad P4: unconnected-(U2-VSSQ4-PadP4) -> /EMMC/GND
- U2 pad P5: unconnected-(U2-VCCQ5-PadP5) -> /EMMC/EMMC_3V3
- U2 pad P6: unconnected-(U2-VSSQ5-PadP6) -> /EMMC/GND
- U3 pad A1: /DDR3_RAM/VDD_DDR -> /STM32MP1_Processor/VDD_DDR
- U3 pad A8: /DDR3_RAM/VDD_DDR -> /STM32MP1_Processor/VDD_DDR
- U3 pad B2: /DDR3_RAM/VDD_DDR -> /STM32MP1_Processor/VDD_DDR
- U3 pad C1: /DDR3_RAM/VDD_DDR -> /STM32MP1_Processor/VDD_DDR
- U3 pad C9: /DDR3_RAM/VDD_DDR -> /STM32MP1_Processor/VDD_DDR
- U3 pad D2: /DDR3_RAM/VDD_DDR -> /STM32MP1_Processor/VDD_DDR
- U3 pad D9: /DDR3_RAM/VDD_DDR -> /STM32MP1_Processor/VDD_DDR
- U3 pad E9: /DDR3_RAM/VDD_DDR -> /STM32MP1_Processor/VDD_DDR
- U3 pad F1: /DDR3_RAM/VDD_DDR -> /STM32MP1_Processor/VDD_DDR
- U3 pad G7: /DDR3_RAM/VDD_DDR -> /STM32MP1_Processor/VDD_DDR
- U3 pad H1: /DDR3_RAM/VREF_DDR -> /STM32MP1_Processor/VDD_DDR
- U3 pad H2: /DDR3_RAM/VDD_DDR -> /STM32MP1_Processor/VDD_DDR
- U3 pad H9: /DDR3_RAM/VDD_DDR -> /STM32MP1_Processor/VDD_DDR
- U3 pad K2: /DDR3_RAM/VDD_DDR -> /STM32MP1_Processor/VDD_DDR
- U3 pad K8: /DDR3_RAM/VDD_DDR -> /STM32MP1_Processor/VDD_DDR
- U3 pad M8: /DDR3_RAM/VREF_DDR -> /STM32MP1_Processor/VDD_DDR
- U3 pad N1: /DDR3_RAM/VDD_DDR -> /STM32MP1_Processor/VDD_DDR
- U3 pad N9: /DDR3_RAM/VDD_DDR -> /STM32MP1_Processor/VDD_DDR
- U3 pad R1: /DDR3_RAM/VDD_DDR -> /STM32MP1_Processor/VDD_DDR
- U3 pad R9: /DDR3_RAM/VDD_DDR -> /STM32MP1_Processor/VDD_DDR
Routing:
- net /DDR3_RAM/DDR_DQ14: track 21.0 -> 0.00 mm
- net /DDR3_RAM/DDR_DQ15: track 19.0 -> 0.00 mm
- net /DDR3_RAM/DDR_CTRL9: track 18.8 -> 0.00 mm
- net /DDR3_RAM/DDR_DQ11: track 15.1 -> 0.00 mm
- net /DDR3_RAM/DDR_A7: track 13.1 -> 0.00 mm, vias 2 -> 0
- net /DDR3_RAM/DDR_CTRL12: track 12.7 -> 0.00 mm
- net /DDR3_RAM/DDR_CTRL3: track 12.6 -> 0.00 mm, vias 2 -> 0
- net /DDR3_RAM/DDR_A11: track 11.7 -> 0.00 mm, vias 2 -> 0
- net /DDR3_RAM/DDR_A14: track 9.31 -> 0.00 mm, vias 2 -> 0
- net /DDR3_RAM/DDR_A13: track 9.26 -> 0.00 mm, vias 2 -> 0
- net /DDR3_RAM/DDR_DQ13: track 9.03 -> 0.00 mm
- net /DDR3_RAM/DDR_BA2: track 9.00 -> 0.00 mm, vias 1 -> 0
- net /DDR3_RAM/DDR_DQ8: track 8.92 -> 0.00 mm
- net /DDR3_RAM/DDR_DQ12: track 8.78 -> 0.00 mm, vias 1 -> 0
- net /DDR3_RAM/DDR_DQ4: track 8.57 -> 0.00 mm, vias 1 -> 0
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
Commit message: Added PMIC, WIFI and updated to STM32MP157 design
Parts:
- added C10: 100nF, Capacitor_SMD:C_0402_1005Metric, F.Cu at (177.9, 131.3)
- added C11: 100nF, Capacitor_SMD:C_0402_1005Metric, F.Cu at (177.9, 133.3)
- added C12: 100nF, Capacitor_SMD:C_0402_1005Metric, F.Cu at (180.8, 127.4)
- added C13: 10uF, Capacitor_SMD:C_0402_1005Metric, F.Cu at (180.8, 129.3)
- added C14: 10uF, Capacitor_SMD:C_0402_1005Metric, F.Cu at (180.8, 131.3)
- added C15: 100nF, Capacitor_SMD:C_0402_1005Metric, F.Cu at (180.8, 133.3)
- added C16: 100nF, Capacitor_SMD:C_0402_1005Metric, F.Cu at (183.7, 127.4)
- added C17: 100nF, Capacitor_SMD:C_0402_1005Metric, F.Cu at (183.7, 129.3)
- added C18: 10uF, Capacitor_SMD:C_0402_1005Metric, F.Cu at (183.7, 131.3)
- added C19: 10uF, Capacitor_SMD:C_0402_1005Metric, F.Cu at (183.7, 133.3)
- added C20: 10uF, Capacitor_SMD:C_0402_1005Metric, F.Cu at (213.6, 110.7)
- added C21: 100nF, Capacitor_SMD:C_0402_1005Metric, F.Cu at (213.6, 112.7)
- added C22: 2.7pF, Capacitor_SMD:C_0402_1005Metric, F.Cu at (213.6, 114.7)
- added C23: 2.7pF, Capacitor_SMD:C_0805_2012Metric, F.Cu at (214.4, 117.2)
- added C24: 10uF, Capacitor_SMD:C_0402_1005Metric, F.Cu at (221.9, 94.4)
- added C25: 100nF, Capacitor_SMD:C_0402_1005Metric, F.Cu at (221.9, 96.3)
- added C26: 100nF, Capacitor_SMD:C_0402_1005Metric, F.Cu at (221.9, 98.3)
- added C27: 100nF, Capacitor_SMD:C_0402_1005Metric, F.Cu at (221.9, 100.3)
- added C28: 100nF, Capacitor_SMD:C_0402_1005Metric, F.Cu at (221.9, 102.2)
- added C29: 2.2uF, Capacitor_SMD:C_0402_1005Metric, F.Cu at (221.9, 104.2)
- added C30: 10uF, Capacitor_SMD:C_0402_1005Metric, F.Cu at (221.9, 106.2)
- added C31: 100nF, Capacitor_SMD:C_0402_1005Metric, F.Cu at (202.2, 140.7)
- added C32: 10uF, Capacitor_SMD:C_0402_1005Metric, F.Cu at (202.2, 142.7)
- added C33: 100nF, Capacitor_SMD:C_0402_1005Metric, F.Cu at (202.2, 144.7)
- added C34: 10uF, Capacitor_SMD:C_0402_1005Metric, F.Cu at (202.2, 146.7)
- added C35: 100nF, Capacitor_SMD:C_0402_1005Metric, F.Cu at (202.2, 148.6)
- added C36: 10pF, Capacitor_SMD:C_0402_1005Metric, F.Cu at (202.2, 150.6)
- added C37: 10pF, Capacitor_SMD:C_0402_1005Metric, F.Cu at (205.0, 140.7)
- added C38: 10pF, Capacitor_SMD:C_0402_1005Metric, F.Cu at (205.0, 142.7)
- added C39: 10pF, Capacitor_SMD:C_0402_1005Metric, F.Cu at (205.0, 144.7)
- added C4: 100nF, Capacitor_SMD:C_0402_1005Metric, F.Cu at (175.1, 127.4)
- added C40: 27pF, Capacitor_SMD:C_0402_1005Metric, F.Cu at (205.0, 146.7)
- added C41: 27pF, Capacitor_SMD:C_0402_1005Metric, F.Cu at (205.0, 148.6)
- added C42: 100nF, Capacitor_SMD:C_0402_1005Metric, F.Cu at (205.0, 150.6)
- added C43: 470pF, Capacitor_SMD:C_0402_1005Metric, F.Cu at (207.9, 140.7)
- added C44: 1uF, Capacitor_SMD:C_0402_1005Metric, F.Cu at (207.9, 142.7)
- added C45: 22nf, Capacitor_SMD:C_0402_1005Metric, F.Cu at (207.9, 144.7)
- added C46: 100uF, Capacitor_SMD:C_0402_1005Metric, F.Cu at (189.6, 113.4)
- added C47: 1uF, Capacitor_SMD:C_0402_1005Metric, F.Cu at (189.6, 115.4)
- added C48: 100nF, Capacitor_SMD:C_0402_1005Metric, F.Cu at (189.6, 117.4)
- added C49: 100nF, Capacitor_SMD:C_0402_1005Metric, F.Cu at (189.6, 119.3)
- added C5: 100nF, Capacitor_SMD:C_0402_1005Metric, F.Cu at (175.1, 129.3)
- added C50: 100nF, Capacitor_SMD:C_0402_1005Metric, F.Cu at (189.6, 121.3)
- added C51: 1uF, Capacitor_SMD:C_0402_1005Metric, F.Cu at (192.5, 113.4)
- added C52: 100nF, Capacitor_SMD:C_0402_1005Metric, F.Cu at (192.5, 115.4)
- added C53: 100nF, Capacitor_SMD:C_0402_1005Metric, F.Cu at (192.5, 117.4)
- added C54: 4.7uF, Capacitor_SMD:C_0402_1005Metric, F.Cu at (192.5, 119.3)
- added C55: 100nF, Capacitor_SMD:C_0402_1005Metric, F.Cu at (192.5, 121.3)
- added C56: 100nF, Capacitor_SMD:C_0402_1005Metric, F.Cu at (195.4, 113.4)
- added C57: 100nF, Capacitor_SMD:C_0402_1005Metric, F.Cu at (195.4, 115.4)
- added C58: 10pF, Capacitor_SMD:C_0402_1005Metric, F.Cu at (195.4, 117.4)
- added C59: 1uF, Capacitor_SMD:C_0402_1005Metric, F.Cu at (87.1, 76.7)
- added C6: 100nF, Capacitor_SMD:C_0402_1005Metric, F.Cu at (175.1, 131.3)
- added C60: 1uF, Capacitor_SMD:C_0402_1005Metric, F.Cu at (87.1, 78.6)
- added C61: 1uF, Capacitor_SMD:C_0402_1005Metric, F.Cu at (87.1, 80.6)
- added C62: 1uF, Capacitor_SMD:C_0402_1005Metric, F.Cu at (87.1, 82.6)
- added C63: 1uF, Capacitor_SMD:C_0402_1005Metric, F.Cu at (87.1, 84.5)
- added C64: 1uF, Capacitor_SMD:C_0402_1005Metric, F.Cu at (87.1, 86.5)
- added C65: 1uF, Capacitor_SMD:C_0402_1005Metric, F.Cu at (87.1, 88.5)
- added C66: 1uF, Capacitor_SMD:C_0402_1005Metric, F.Cu at (87.1, 90.5)
- added C7: 10uF, Capacitor_SMD:C_0402_1005Metric, F.Cu at (175.1, 133.3)
- added C8: 10uF, Capacitor_SMD:C_0402_1005Metric, F.Cu at (177.9, 127.4)
- added C9: 10uF, Capacitor_SMD:C_0402_1005Metric, F.Cu at (177.9, 129.3)
- added D1: ESD9B5.0ST5G, Diode_SMD:D_SOD-923, F.Cu at (210.9, 110.7)
- added D10: SMF54A, Diode_SMD:D_SMF, F.Cu at (195.6, 101.1)
- added D11: ESD9B3.3ST5G, Diode_SMD:D_SOD-923, F.Cu at (194.1, 108.3)
- added D2: ESD9B5.0ST5G, Diode_SMD:D_SOD-923, F.Cu at (210.9, 112.7)
- added D3: ESD9B5.0ST5G, Diode_SMD:D_SOD-923, F.Cu at (210.9, 114.6)
- added D4: ESD9B5.0ST5G, Diode_SMD:D_SOD-923, F.Cu at (210.9, 116.6)
- added D5: ESD9B5.0ST5G, Diode_SMD:D_SOD-923, F.Cu at (210.9, 118.5)
- added D6: ESD9B5.0ST5G, Diode_SMD:D_SOD-923, F.Cu at (210.9, 120.5)
- added D7: ESD9B5.0ST5G, Diode_SMD:D_SOD-923, F.Cu at (210.9, 122.4)
- added D8: ESD9B3.3ST5G, Diode_SMD:D_SOD-923, F.Cu at (217.8, 148.6)
- added D9: ESD9B3.3ST5G, Diode_SMD:D_SOD-923, F.Cu at (217.8, 150.6)
- added FB1: FerriteBead_Small, Inductor_SMD:L_Walsin_WLFM252009x, F.Cu at (221.7, 143.1)
- added FB2: FerriteBead_Small, Inductor_SMD:L_Walsin_WLFM252009x, F.Cu at (221.7, 146.7)
- added J2: Conn_Coaxial_x2_Isolated, Connector_Coaxial:U.FL_Molex_MCRF_73412-0110_Vertical, F.Cu at (195.7, 96.5)
- added R100: 10K, Resistor_SMD:R_0402_1005Metric, F.Cu at (186.7, 119.4)
- added R101: 10K, Resistor_SMD:R_0402_1005Metric, F.Cu at (186.7, 121.4)
- added R102: 0R, Resistor_SMD:R_0402_1005Metric, F.Cu at (186.7, 123.4)
- added R30: 100R, Resistor_SMD:R_0402_1005Metric, F.Cu at (175.1, 135.2)
- added R31: 33R, Resistor_SMD:R_0402_1005Metric, F.Cu at (202.2, 114.7)
- added R32: 33R, Resistor_SMD:R_0402_1005Metric, F.Cu at (202.2, 116.7)
- added R33: 33R, Resistor_SMD:R_0402_1005Metric, F.Cu at (202.2, 118.7)
- added R34: 33R, Resistor_SMD:R_0402_1005Metric, F.Cu at (205.1, 110.8)
- added R35: 10K, Resistor_SMD:R_0402_1005Metric, F.Cu at (205.1, 112.7)
- added R36: 10K, Resistor_SMD:R_0402_1005Metric, F.Cu at (205.1, 114.7)
- added R37: 10K, Resistor_SMD:R_0402_1005Metric, F.Cu at (205.1, 116.7)
- added R38: 10K, Resistor_SMD:R_0402_1005Metric, F.Cu at (205.1, 118.7)
- added R39: 10K, Resistor_SMD:R_0402_1005Metric, F.Cu at (208.0, 110.8)
- added R40: 10K, Resistor_SMD:R_0402_1005Metric, F.Cu at (208.0, 112.7)
- added R41: 10K, Resistor_SMD:R_0402_1005Metric, F.Cu at (208.0, 114.7)
- added R42: 0R, Resistor_SMD:R_0402_1005Metric, F.Cu at (208.0, 116.7)
- added R43: 0R, Resistor_SMD:R_0402_1005Metric, F.Cu at (224.8, 94.4)
- added R44: 0R, Resistor_SMD:R_0402_1005Metric, F.Cu at (224.8, 96.4)
- added R45: 0R, Resistor_SMD:R_0402_1005Metric, F.Cu at (213.8, 126.4)
- added R46: 0R, Resistor_SMD:R_0402_1005Metric, F.Cu at (213.8, 128.4)
- added R47: 0R, Resistor_SMD:R_0402_1005Metric, F.Cu at (213.8, 130.4)
- added R48: 10K, Resistor_SMD:R_0402_1005Metric, F.Cu at (213.8, 132.4)
- added R49: 10K, Resistor_SMD:R_0402_1005Metric, F.Cu at (213.8, 134.4)
- added R50: 10K, Resistor_SMD:R_0402_1005Metric, F.Cu at (213.8, 136.3)
- added R51: 10K, Resistor_SMD:R_0402_1005Metric, F.Cu at (213.8, 138.3)
- added R52: 10K, Resistor_SMD:R_0402_1005Metric, F.Cu at (213.8, 140.3)
- added R53: 10K, Resistor_SMD:R_0402_1005Metric, F.Cu at (216.8, 126.4)
- added R54: 10K, Resistor_SMD:R_0402_1005Metric, F.Cu at (216.8, 128.4)
- added R55: 0R, Resistor_SMD:R_0402_1005Metric, F.Cu at (216.8, 130.4)
- added R56: 0R, Resistor_SMD:R_0402_1005Metric, F.Cu at (216.8, 132.4)
- added R57: 10K, Resistor_SMD:R_0402_1005Metric, F.Cu at (216.8, 134.4)
- added R58: 33R, Resistor_SMD:R_0402_1005Metric, F.Cu at (216.8, 136.3)
- added R59: 33R, Resistor_SMD:R_0402_1005Metric, F.Cu at (216.8, 138.3)
- added R60: 33R, Resistor_SMD:R_0402_1005Metric, F.Cu at (216.8, 140.3)
- added R61: 33R, Resistor_SMD:R_0402_1005Metric, F.Cu at (219.7, 126.4)
- added R62: 33R, Resistor_SMD:R_0402_1005Metric, F.Cu at (219.7, 128.4)
- added R63: 10R, Resistor_SMD:R_0402_1005Metric, F.Cu at (219.7, 130.4)
- added R64: 0R, Resistor_SMD:R_0402_1005Metric, F.Cu at (219.7, 132.4)
- added R65: 0R, Resistor_SMD:R_0402_1005Metric, F.Cu at (219.7, 134.4)
- added R66: 33R, Resistor_SMD:R_0402_1005Metric, F.Cu at (219.7, 136.3)
- added R67: 1.5K, Resistor_SMD:R_0402_1005Metric, F.Cu at (219.7, 138.3)
- added R68: 12.1K, Resistor_SMD:R_0402_1005Metric, F.Cu at (219.7, 140.3)
- added R69: 49.9, Resistor_SMD:R_0402_1005Metric, F.Cu at (222.6, 126.4)
- added R70: 49.9, Resistor_SMD:R_0402_1005Metric, F.Cu at (222.6, 128.4)
- added R71: 49.9, Resistor_SMD:R_0402_1005Metric, F.Cu at (222.6, 130.4)
- added R72: 49.9, Resistor_SMD:R_0402_1005Metric, F.Cu at (222.6, 132.4)
- added R73: 0R, Resistor_SMD:R_0402_1005Metric, F.Cu at (175.1, 113.4)
- added R74: 0R, Resistor_SMD:R_0402_1005Metric, F.Cu at (175.1, 115.4)
- added R75: 10K, Resistor_SMD:R_0402_1005Metric, F.Cu at (175.1, 117.4)
- added R76: 10K, Resistor_SMD:R_0402_1005Metric, F.Cu at (175.1, 119.4)
- added R77: 10K, Resistor_SMD:R_0402_1005Metric, F.Cu at (175.1, 121.4)
- added R78: 10K, Resistor_SMD:R_0402_1005Metric, F.Cu at (175.1, 123.4)
- added R79: 10K, Resistor_SMD:R_0402_1005Metric, F.Cu at (178.0, 113.4)
- added R80: 10K, Resistor_SMD:R_0402_1005Metric, F.Cu at (178.0, 115.4)
- added R81: 0R, Resistor_SMD:R_0402_1005Metric, F.Cu at (178.0, 117.4)
- added R82: 0R, Resistor_SMD:R_0402_1005Metric, F.Cu at (178.0, 119.4)
- added R83: 0R, Resistor_SMD:R_0402_1005Metric, F.Cu at (178.0, 121.4)
- added R84: 0R, Resistor_SMD:R_0402_1005Metric, F.Cu at (178.0, 123.4)
- added R85: 0R, Resistor_SMD:R_0402_1005Metric, F.Cu at (180.9, 113.4)
- added R86: 0R, Resistor_SMD:R_0402_1005Metric, F.Cu at (180.9, 115.4)
- added R87: 0R, Resistor_SMD:R_0402_1005Metric, F.Cu at (180.9, 117.4)
- added R88: 0R, Resistor_SMD:R_0402_1005Metric, F.Cu at (180.9, 119.4)
- added R89: 10K, Resistor_SMD:R_0402_1005Metric, F.Cu at (180.9, 121.4)
- added R90: 10K, Resistor_SMD:R_0402_1005Metric, F.Cu at (180.9, 123.4)
- added R91: 0R, Resistor_SMD:R_0402_1005Metric, F.Cu at (183.8, 113.4)
- added R92: 0R, Resistor_SMD:R_0402_1005Metric, F.Cu at (183.8, 115.4)
- added R93: 0R, Resistor_SMD:R_0402_1005Metric, F.Cu at (183.8, 117.4)
- added R94: 0R, Resistor_SMD:R_0402_1005Metric, F.Cu at (183.8, 119.4)
- added R95: 0R, Resistor_SMD:R_0402_1005Metric, F.Cu at (183.8, 121.4)
- added R96: 0R, Resistor_SMD:R_0402_1005Metric, F.Cu at (183.8, 123.4)
- added R97: 0R, Resistor_SMD:R_0402_1005Metric, F.Cu at (186.7, 113.4)
- added R98: 0R, Resistor_SMD:R_0402_1005Metric, F.Cu at (186.7, 115.4)
- added R99: 0R, Resistor_SMD:R_0402_1005Metric, F.Cu at (186.7, 117.4)
- added TR1: PT61017PEL, Transformer_SMD:Transformer_Ethernet_Bourns_PT61017PEL, F.Cu at (204.7, 131.7)
- added U4: LAN8742A, Package_DFN_QFN:VQFN-24-1EP_4x4mm_P0.5mm_EP2.5x2.5mm_ThermalVias, F.Cu at (215.9, 144.5)
- added U5: KC2520Z, Oscillator:Oscillator_SMD_Kyocera_KC2520Z-4Pin_2.5x2.0mm, F.Cu at (214.4, 149.9)
- added U6: FC905AAAMD, FC905AAAMD:XCVR_FC905AAAMD, F.Cu at (183.2, 102.9)
- added U7: STM32MP157DACx, Package_BGA:ST_TFBGA-361_12x12mm_Layout23x23_P0.5mmP0.65mm, F.Cu at (96.0, 83.2)
- added Y1: abr-asek-1-32768khz, Oscillator:Oscillator_SMD_Abracon_ASE-4Pin_3.2x2.5mm, F.Cu at (195.3, 105.1)
- R28: value 10K -> 33R
- moved R26 76.9 mm to (202.2, 110.8)
- moved R28 71.9 mm to (202.2, 112.7)
- moved J1 46.3 mm to (211.0, 80.5)
Connections:
- J1 pad 1: unconnected-(J1-DAT2-Pad1) -> Net-(D1-A2)
- J1 pad 2: unconnected-(J1-DAT3/CD-Pad2) -> Net-(D2-A2)
- J1 pad 3: unconnected-(J1-CMD-Pad3) -> Net-(D3-A2)
- J1 pad 4: unconnected-(J1-VDD-Pad4) -> Net-(J1-VDD)
- J1 pad 5: unconnected-(J1-CLK-Pad5) -> /SD_CARD/uSD_BUS5
- J1 pad 6: unconnected-(J1-VSS-Pad6) -> /SD_CARD/GND
- J1 pad 7: unconnected-(J1-DAT0-Pad7) -> Net-(D5-A2)
- J1 pad 8: unconnected-(J1-DAT1-Pad8) -> Net-(D6-A2)
- J1 pad 9: unconnected-(J1-DET-Pad9) -> Net-(D7-A2)
- R26 pad 1: /EMMC/EMMC10 -> Net-(D1-A2)
- R26 pad 2: /EMMC/EMMC_DS -> /SD_CARD/uSD_BUS2
- R27 pad 1: /EMMC/EMMC11 -> /EMMC/EMMC10
- R28 pad 1: /EMMC/EMMC_3V3 -> Net-(D2-A2)
- R28 pad 2: /EMMC/EMMC_DS -> /SD_CARD/uSD_BUS3
- U1 pad AA2: unconnected-(U1-PB11-PadAA2) -> /Ethernet/RMII2
- U1 pad AA3: unconnected-(U1-PA1-PadAA3) -> /STM32MP1_Processor/RMII_REFCLK
- U1 pad AA7: unconnected-(U1-PC5-PadAA7) -> /Ethernet/RMII4
- U1 pad AA9: unconnected-(U1-PG13-PadAA9) -> /Ethernet/RMII0
- U1 pad V3: unconnected-(U1-PG2-PadV3) -> /Ethernet/RMII7
- U1 pad W1: unconnected-(U1-PG3-PadW1) -> /STM32MP1_Processor/RMII_NRST
- U1 pad Y10: unconnected-(U1-PG14-PadY10) -> /Ethernet/RMII1
- U1 pad Y11: /EMMC/EMMC11 -> /EMMC/EMMC10
- U1 pad Y4: unconnected-(U1-PA2-PadY4) -> /Ethernet/RMII6
- U1 pad Y7: unconnected-(U1-PC4-PadY7) -> /Ethernet/RMII3
- U1 pad Y9: unconnected-(U1-PC1-PadY9) -> /STM32MP1_Processor/RMII_CRS_DV
- U2 pad C2: unconnected-(U2-VDDI-PadC2) -> Net-(U2-VDDI)
- U2 pad H5: /EMMC/EMMC_DS -> unconnected-(U2-DS-PadH5)
